File: Hardware/PCB/psu.kicad_sch (KiCad schematic)
At the start: 41 parts, among them J19 12V IN, Q3 IRF740, Q82 IRF740, Q83 IRF740, Q84 BC556, U22 IR2153, U23 SY317, U24 AMS1117-3.3, U25 MC34063AP

Commit message: schematic update
Parts:
- renumbered C34 to C17, C37 to C18, C38 to C19, C39 to C20, C40 to C21, C41 to C22, C42 to C23, C43 to C24, C44 to C25, C48 to C26, C49 to C27, C31 to C28, C32 to C29, C33 to C30, C45 to C31, C35 to C32, C36 to C33, C46 to C34, C47 to C35, D5 to D2, D6 to D3, D7 to D4, D8 to D5, J19 to J22, L2 to L1, Q82 to Q85, Q83 to Q86, Q3 to Q87, Q84 to Q88, R110 to R114, R108 to R115, R111 to R116, R113 to R117, R109 to R118, R112 to R119, R114 to R120, R115 to R121, U22 to U25, U25 to U26
Other:
- moved on the sheet: C26, C27

Commit message: Hardware Update Schematic Done Placement started
Parts:
- removed C18, C21: 4µ7, Capacitor_SMD:C_0805_2012Metric, symbol Device:C
- removed C19, C20: 100n, Capacitor_SMD:C_0805_2012Metric, symbol Device:C
- removed C28, C29, C32, C33: 22µ, symbol Device:C
- removed D2, D3: BAT41, Diode_THT:D_DO-35_SOD27_P7.62mm_Horizontal, symbol Diode:BAT41
- removed J22: 12V IN, symbol Connector_Generic:Conn_01x02
- added C1, C2, C3, C4: 22µ 250V, Capacitor_THT:CP_Radial_D10.0mm_P5.00mm, symbol Device:C_Polarized
- added D401, D402: 1N4007, Diode_THT:D_DO-41_SOD81_P10.16mm_Horizontal, symbol Diode:1N4007
- added J401: Barrel_Jack, Connector_BarrelJack:BarrelJack_Horizontal, symbol Connector:Barrel_Jack
- C401: renamed from C17; footprint (none) -> Capacitor_THT:CP_Radial_D5.0mm_P2.50mm
- C410: renamed from C26; footprint (none) -> Capacitor_THT:C_Disc_D3.0mm_W1.6mm_P2.50mm
- C411: renamed from C27; footprint (none) -> Capacitor_THT:C_Disc_D3.0mm_W1.6mm_P2.50mm
- C414: renamed from C30; footprint (none) -> Capacitor_THT:C_Rect_L18.0mm_W8.0mm_P15.00mm_FKS3_FKP3
- C415: renamed from C31; footprint (none) -> Capacitor_THT:C_Disc_D3.0mm_W1.6mm_P2.50mm
- C418: renamed from C34; footprint (none) -> Capacitor_THT:C_Disc_D3.0mm_W1.6mm_P2.50mm
- C419: renamed from C35; footprint (none) -> Capacitor_THT:C_Disc_D3.0mm_W1.6mm_P2.50mm
- Q404: renamed from Q88; footprint Package_TO_SOT_THT:TO-92_Inline -> Package_TO_SOT_THT:TO-92
- R401: renamed from R114; footprint (none) -> Resistor_THT:R_Axial_DIN0207_L6.3mm_D2.5mm_P2.54mm_Vertical
- R402: renamed from R115; footprint (none) -> Resistor_THT:R_Axial_DIN0614_L14.3mm_D5.7mm_P5.08mm_Vertical
- R403: renamed from R116; footprint (none) -> Resistor_THT:R_Axial_DIN0207_L6.3mm_D2.5mm_P2.54mm_Vertical
- R404: renamed from R117; footprint (none) -> Resistor_THT:R_Axial_DIN0207_L6.3mm_D2.5mm_P2.54mm_Vertical
- R405: renamed from R118; footprint (none) -> Resistor_THT:R_Axial_DIN0207_L6.3mm_D2.5mm_P2.54mm_Vertical
- R406: renamed from R119; footprint (none) -> Resistor_THT:R_Axial_DIN0207_L6.3mm_D2.5mm_P2.54mm_Vertical
- R407: renamed from R120; footprint (none) -> Resistor_THT:R_Axial_DIN0207_L6.3mm_D2.5mm_P2.54mm_Vertical
- R408: renamed from R121; footprint (none) -> Resistor_THT:R_Axial_DIN0207_L6.3mm_D2.5mm_P2.54mm_Vertical
- U401: renamed from U23; footprint Package_TO_SOT_SMD:TO-252-2 -> Package_TO_SOT_THT:TO-220-3_Vertical
- U403: renamed from U25; footprint (none) -> Package_DIP:DIP-8_W7.62mm
- renumbered C22 to C406, C23 to C407, C24 to C408, C25 to C409, D4 to D403, D5 to D404, L1 to L401, Q85 to Q401, Q86 to Q402, Q87 to Q403, U24 to U402, U26 to U404
Connections:
- net +12V: now also J401.1
- net +180V: now also C2.1, D402.1 (K)
- net +90V: now also C3.1, C4.1, D401.2 (A)
- net GND: now also C2.2, C3.2, C4.2, J401.2
- net at C414.2, Q401.3 (S), Q402.2 (D)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: now also C1.2
- new net: C1.1, D401.1 (K), D402.2 (A)

Commit message: PCB update finished placing and routing Cleanup Passes need to be done Silkscreen needs to be done
Parts:
- D401, D402, D403: value 1N4007 -> UF4007
Changed lines of the file:
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@@
 			)
 		)
-		(property "Value" "1N4007"
+		(property "Value" "UF4007"
 			(at 262.89 109.22 0)
 			(effects
@@
 			)
 		)
-		(property "Value" "1N4007"
+		(property "Value" "UF4007"
 			(at 243.84 109.22 0)
 			(effects
@@
 			)
 		)
-		(property "Value" "1N4007"
+		(property "Value" "UF4007"
 			(at 102.87 125.73 0)
 			(effects

Commit message: small bugfix update
Parts:
- added D405: UF4007, Diode_THT:D_DO-41_SOD81_P10.16mm_Horizontal, symbol Diode:1N4007
Connections:
- net +12V: now also D405.2 (A)
- net +90V: no longer C414.1, U403.8 (VB)
- new net: C414.1, D405.1 (K), U403.8 (VB)
Other:
- moved on the sheet: C414
Changed lines of the file:
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@@
 	)
 	(junction
+		(at 205.74 119.38)
+		(diameter 0)
+		(color 0 0 0 0)
+	)
+	(junction
 		(at 57.15 44.45)
 		(diameter 0)
@@
 	)
 	(junction
-		(at 223.52 48.26)
+		(at 191.77 111.76)
 		(diameter 0)
 		(color 0 0 0 0)
 	)
 	(junction
-		(at 210.82 128.27)
+		(at 223.52 48.26)
 		(diameter 0)
 		(color 0 0 0 0)
@@
 	)
 	(junction
-		(at 57.15 62.23)
+		(at 205.74 132.08)
 		(diameter 0)
 		(color 0 0 0 0)
 	)
 	(junction
-		(at 205.74 115.57)
+		(at 57.15 62.23)
 		(diameter 0)
 		(color 0 0 0 0)
@@
 	(wire
 		(pts
+			(xy 191.77 111.76) (xy 191.77 114.3)
+		)
+		(stroke
+			(width 0)
+			(type default)
+		)
+	)
+	(wire
+		(pts
 			(xy 58.42 129.54) (xy 62.23 129.54)
 		)
@@
 	(wire
 		(pts
+			(xy 205.74 132.08) (xy 199.39 132.08)
+		)
+		(stroke
+			(width 0)
+			(type default)
+		)
+	)
+	(wire
+		(pts
 			(xy 210.82 128.27) (xy 233.68 128.27)
 		)
@@
 	(wire
 		(pts
-			(xy 191.77 109.22) (xy 191.77 114.3)
+			(xy 191.77 109.22) (xy 191.77 111.76)
 		)
 		(stroke
@@
 	(wire
 		(pts
+			(xy 205.74 132.08) (xy 210.82 132.08)
+		)
+		(stroke
+			(width 0)
+			(type default)
+		)
+	)
+	(wire
+		(pts
 			(xy 121.92 129.54) (xy 121.92 146.05)
 		)
@@
 	(wire
 		(pts
-			(xy 210.82 125.73) (xy 210.82 128.27)
+			(xy 205.74 130.81) (xy 205.74 132.08)
 		)
 		(stroke
@@
 	(wire
 		(pts
+			(xy 205.74 111.76) (xy 201.93 111.76)
+		)
+		(stroke
+			(width 0)
+			(type default)
+		)
+	)
+	(wire
+		(pts
 			(xy 177.8 48.26) (xy 187.96 48.26)
 		)
@@
 	(wire
 		(pts
-			(xy 205.74 115.57) (xy 205.74 119.38)
+			(xy 205.74 111.76) (xy 205.74 119.38)
 		)
 		(stroke
@@
 	(wire
 		(pts
-			(xy 210.82 118.11) (xy 210.82 115.57)
+			(xy 205.74 123.19) (xy 205.74 119.38)
 		)
 		(stroke
@@
 	(wire
 		(pts
-			(xy 210.82 115.57) (xy 205.74 115.57)
-		)
-		(stroke
-			(width 0)
-			(type default)
-		)
-	)
-	(wire
-		(pts
 			(xy 57.15 45.72) (xy 57.15 44.45)
 		)
@@
 	(wire
 		(pts
-			(xy 210.82 132.08) (xy 199.39 132.08)
-		)
-		(stroke
-			(width 0)
-			(type default)
-		)
-	)
-	(wire
-		(pts
 			(xy 184.15 132.08) (xy 180.34 132.08)
 		)
@@
 	(wire
 		(pts
+			(xy 194.31 111.76) (xy 191.77 111.76)
+		)
+		(stroke
+			(width 0)
+			(type default)
+		)
+	)
+	(wire
+		(pts
 			(xy 223.52 55.88) (xy 223.52 48.26)
 		)
@@
 	(wire
 		(pts
-			(xy 205.74 109.22) (xy 205.74 115.57)
-		)
-		(stroke
-			(width 0)
-			(type default)
-		)
-	)
-	(wire
-		(pts
 			(xy 205.74 119.38) (xy 199.39 119.38)
 		)
@@
 	(symbol
 		(lib_id "Device:C")
-		(at 210.82 121.92 0)
+		(at 205.74 127 0)
 		(unit 1)
 		(exclude_from_sim no)
@@
 		(dnp no)
 		(property "Reference" "C414"
-			(at 207.772 119.38 0)
+			(at 200.406 124.714 0)
 			(effects
 				(font
@@
 		)
 		(property "Value" "1µ"
-			(at 207.518 124.46 0)
+			(at 202.438 129.54 0)
 			(effects
 				(font
@@
 		)
 		(property "Footprint" "Capacitor_THT:C_Rect_L18.0mm_W8.0mm_P15.00mm_FKS3_FKP3"
-			(at 211.7852 125.73 0)
+			(at 206.7052 130.81 0)
 			(effects
 				(font
@@
 		)
 		(property "Datasheet" "~"
-			(at 210.82 121.92 0)
+			(at 205.74 127 0)
 			(effects
 				(font
@@
 		)
 		(property "Description" "Unpolarized capacitor"
-			(at 210.82 121.92 0)
+			(at 205.74 127 0)
 			(effects
 				(font
@@
 	)
 	(symbol
-		(lib_id "power:+VSW")
-		(at 205.74 109.22 0)
-		(unit 1)
-		(exclude_from_sim no)
-		(in_bom yes)
-		(on_board yes)
-		(dnp no)
-		(fields_autoplaced yes)
-		(property "Reference" "#PWR0425"
-			(at 205.74 113.03 0)
-			(effects
-				(font
-					(size 1.27 1.27)
-				)
-				(hide yes)
-			)
-		)
-		(property "Value" "+90V"
-			(at 205.74 104.14 0)
-			(effects
-				(font
-					(size 1.27 1.27)
-				)
-			)
-		)
-		(property "Footprint" ""
-			(at 205.74 109.22 0)
-			(effects
-				(font
-					(size 1.27 1.27)
-				)
-				(hide yes)
-			)
-		)
-		(property "Datasheet" ""
-			(at 205.74 109.22 0)
-			(effects
-				(font
-					(size 1.27 1.27)
-				)
-				(hide yes)
-			)
-		)
-		(property "Description" "Power symbol creates a global label with name \"+VSW\""
-			(at 205.74 109.22 0)
-			(effects
-				(font
-					(size 1.27 1.27)
-				)
-				(hide yes)
-			)
-		)
-		(pin "1"
-		)
-		(instances
-			(project "nixie"
-				(path "/36badbe3-7abc-48d5-8c49-5ac646d9041f/ffec0fe8-35a1-4ab6-b4ec-cde8cf0800bc"
-					(reference "#PWR0425")
-					(unit 1)
-				)
-			)
-		)
-	)
-	(symbol
 		(lib_id "Device:L")
 		(at 73.66 129.54 90)
@@
 	)
 	(symbol
+		(lib_id "Diode:1N4007")
+		(at 198.12 111.76 0)
+		(mirror y)
+		(unit 1)
+		(exclude_from_sim no)
+		(in_bom yes)
+		(on_board yes)
+		(dnp no)
+		(fields_autoplaced yes)
+		(property "Reference" "D405"
+			(at 198.12 105.41 0)
+			(effects
+				(font
+					(size 1.27 1.27)
+				)
+			)
+		)
+		(property "Value" "UF4007"
+			(at 198.12 107.95 0)
+			(effects
+				(font
+					(size 1.27 1.27)
+				)
+			)
+		)
+		(property "Footprint" "Diode_THT:D_DO-41_SOD81_P10.16mm_Horizontal"
+			(at 198.12 116.205 0)
+			(effects
+				(font
+					(size 1.27 1.27)
+				)
+				(hide yes)
+			)
+		)
+		(property "Datasheet" "http://www.vishay.com/docs/88503/1n4001.pdf"
+			(at 198.12 111.76 0)
+			(effects
+				(font
+					(size 1.27 1.27)
+				)
+				(hide yes)
+			)
+		)
+		(property "Description" "1000V 1A General Purpose Rectifier Diode, DO-41"
+			(at 198.12 111.76 0)
+			(effects
+				(font
+					(size 1.27 1.27)
+				)
+				(hide yes)
+			)
+		)
+		(property "Sim.Device" "D"
+			(at 198.12 111.76 0)
+			(effects
+				(font
+					(size 1.27 1.27)
+				)
+				(hide yes)
+			)
+		)
+		(property "Sim.Pins" "1=K 2=A"
+			(at 198.12 111.76 0)
+			(effects
+				(font
+					(size 1.27 1.27)
+				)
+				(hide yes)
+			)
+		)
+		(pin "2"
+		)
+		(pin "1"
+		)
+		(instances
+			(project "nixie"
+				(path "/36badbe3-7abc-48d5-8c49-5ac646d9041f/ffec0fe8-35a1-4ab6-b4ec-cde8cf0800bc"
+					(reference "D405")
+					(unit 1)
+				)
+			)
+		)
+	)
+	(symbol
 		(lib_id "power:GND")
 		(at 232.41 63.5 0)
@@
 		(on_board yes)
 		(dnp no)
-		(fields_autoplaced yes)
 		(property "Reference" "U403"
-			(at 193.9641 111.76 0)
+			(at 193.04 138.684 0)
 			(effects
 				(font
@@
 		)
 		(property "Value" "IR2153"
-			(at 193.9641 114.3 0)
+			(at 193.04 141.224 0)
 			(effects
 				(font

Commit message: reviewed version from thebrutzler
Parts:
- added R3: 220k, Resistor_THT:R_Axial_DIN0207_L6.3mm_D2.5mm_P2.54mm_Vertical, symbol Device:R
Connections:
- net +180V: now also R3.2
- net GND: now also R3.1
Other:
- moved on the sheet: D404
Changed lines of the file:
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@@
 	(title_block
 		(title "Z5600M Nixie Clock with ESP32")
-		(date "2024-09-16")
-		(rev "1.0")
+		(date "2024-10-04")
+		(rev "1.1")
 		(company "Synthron")
 	)
@@
 	(wire
 		(pts
-			(xy 73.66 142.24) (xy 76.2 142.24)
-		)
-		(stroke
-			(width 0)
-			(type default)
-		)
-	)
-	(wire
-		(pts
 			(xy 210.82 128.27) (xy 210.82 132.08)
 		)
@@
 	(wire
 		(pts
+			(xy 73.66 142.24) (xy 73.66 151.13)
+		)
+		(stroke
+			(width 0)
+			(type default)
+		)
+	)
+	(wire
+		(pts
 			(xy 191.77 109.22) (xy 191.77 111.76)
 		)
@@
 	(wire
 		(pts
-			(xy 271.78 113.03) (xy 266.7 113.03)
+			(xy 266.7 113.03) (xy 271.78 113.03)
 		)
 		(stroke
@@
 	(wire
 		(pts
-			(xy 254 128.27) (xy 233.68 128.27)
+			(xy 205.74 48.26) (xy 207.01 48.26)
 		)
 		(stroke
@@
 	(wire
 		(pts
-			(xy 205.74 48.26) (xy 207.01 48.26)
+			(xy 276.225 126.365) (xy 276.225 113.03)
 		)
 		(stroke
@@
 	(wire
 		(pts
+			(xy 233.68 128.27) (xy 254 128.27)
+		)
+		(stroke
+			(width 0)
+			(type default)
+		)
+	)
+	(wire
+		(pts
 			(xy 77.47 129.54) (xy 93.98 129.54)
 		)
@@
 	(wire
 		(pts
+			(xy 276.225 113.03) (xy 271.78 113.03)
+		)
+		(stroke
+			(width 0)
+			(type default)
+		)
+	)
+	(wire
+		(pts
 			(xy 232.41 45.72) (xy 232.41 48.26)
 		)
@@
 	(wire
 		(pts
+			(xy 276.225 146.05) (xy 276.225 133.985)
+		)
+		(stroke
+			(width 0)
+			(type default)
+		)
+	)
+	(wire
+		(pts
 			(xy 172.72 135.89) (xy 172.72 137.16)
 		)
@@
 	(wire
 		(pts
-			(xy 73.66 151.13) (xy 73.66 142.24)
-		)
-		(stroke
-			(width 0)
-			(type default)
-		)
-	)
-	(wire
-		(pts
 			(xy 172.72 144.78) (xy 172.72 146.05)
 		)
@@
 	(wire
 		(pts
-			(xy 83.82 142.24) (xy 86.36 142.24)
+			(xy 81.28 142.24) (xy 86.36 142.24)
 		)
 		(stroke
@@
 	(symbol
 		(lib_id "Diode:1N4148")
-		(at 80.01 142.24 180)
+		(at 77.47 142.24 180)
 		(unit 1)
 		(exclude_from_sim no)
@@
 		(fields_autoplaced yes)
 		(property "Reference" "D404"
-			(at 80.01 135.89 0)
+			(at 77.47 135.89 0)
 			(effects
 				(font
@@
 		)
 		(property "Value" "1N4148"
-			(at 80.01 138.43 0)
+			(at 77.47 138.43 0)
 			(effects
 				(font
@@
 		)
 		(property "Footprint" "Diode_THT:D_DO-35_SOD27_P7.62mm_Horizontal"
-			(at 80.01 142.24 0)
+			(at 77.47 142.24 0)
 			(effects
 				(font
@@
 		)
 		(property "Datasheet" "https://assets.nexperia.com/documents/data-sheet/1N4148_1N4448.pdf"
-			(at 80.01 142.24 0)
+			(at 77.47 142.24 0)
 			(effects
 				(font
@@
 		)
 		(property "Description" "100V 0.15A standard switching diode, DO-35"
-			(at 80.01 142.24 0)
+			(at 77.47 142.24 0)
 			(effects
 				(font
@@
 		)
 		(property "Sim.Device" "D"
-			(at 80.01 142.24 0)
+			(at 77.47 142.24 0)
 			(effects
 				(font
@@
 		)
 		(property "Sim.Pins" "1=K 2=A"
-			(at 80.01 142.24 0)
+			(at 77.47 142.24 0)
 			(effects
 				(font
@@
 	)
 	(symbol
+		(lib_id "Device:R")
+		(at 276.225 130.175 0)
+		(mirror x)
+		(unit 1)
+		(exclude_from_sim no)
+		(in_bom yes)
+		(on_board yes)
+		(dnp no)
+		(property "Reference" "R3"
+			(at 282.575 130.175 0)
+			(effects
+				(font
+					(size 1.27 1.27)
+				)
+				(justify right)
+			)
+		)
+		(property "Value" "220k"
+			(at 276.225 132.461 90)
+			(effects
+				(font
+					(size 1.27 1.27)
+				)
+				(justify right)
+			)
+		)
+		(property "Footprint" "Resistor_THT:R_Axial_DIN0207_L6.3mm_D2.5mm_P2.54mm_Vertical"
+			(at 274.447 130.175 90)
+			(effects
+				(font
+					(size 1.27 1.27)
+				)
+				(hide yes)
+			)
+		)
+		(property "Datasheet" "~"
+			(at 276.225 130.175 0)
+			(effects
+				(font
+					(size 1.27 1.27)
+				)
+				(hide yes)
+			)
+		)
+		(property "Description" "Resistor"
+			(at 276.225 130.175 0)
+			(effects
+				(font
+					(size 1.27 1.27)
+				)
+				(hide yes)
+			)
+		)
+		(pin "1"
+		)
+		(pin "2"
+		)
+		(instances
+			(project "nixie"
+				(path "/36badbe3-7abc-48d5-8c49-5ac646d9041f/ffec0fe8-35a1-4ab6-b4ec-cde8cf0800bc"
+					(reference "R3")
+					(unit 1)
+				)
+			)
+		)
+	)
+	(symbol
 		(lib_id "Transistor_FET:IRF740")
 		(at 231.14 121.92 0)
@@
 	)
 	(symbol
+		(lib_id "power:GND")
+		(at 276.225 146.05 0)
+		(unit 1)
+		(exclude_from_sim no)
+		(in_bom yes)
+		(on_board yes)
+		(dnp no)
+		(fields_autoplaced yes)
+		(property "Reference" "#PWR03"
+			(at 276.225 152.4 0)
+			(effects
+				(font
+					(size 1.27 1.27)
+				)
+				(hide yes)
+			)
+		)
+		(property "Value" "GND"
+			(at 276.225 151.13 0)
+			(effects
+				(font
+					(size 1.27 1.27)
+				)
+			)
+		)
+		(property "Footprint" ""
+			(at 276.225 146.05 0)
+			(effects
+				(font
+					(size 1.27 1.27)
+				)
+				(hide yes)
+			)
+		)
+		(property "Datasheet" ""
+			(at 276.225 146.05 0)
+			(effects
+				(font
+					(size 1.27 1.27)
+				)
+				(hide yes)
+			)
+		)
+		(property "Description" "Power symbol creates a global label with name \"GND\" , ground"
+			(at 276.225 146.05 0)
+			(effects
+				(font
+					(size 1.27 1.27)
+				)
+				(hide yes)
+			)
+		)
+		(pin "1"
+		)
+		(instances
+			(project "nixie"
+				(path "/36badbe3-7abc-48d5-8c49-5ac646d9041f/ffec0fe8-35a1-4ab6-b4ec-cde8cf0800bc"
+					(reference "#PWR03")
+					(unit 1)
+				)
+			)
+		)
+	)
+	(symbol
 		(lib_id "Device:R")
 		(at 73.66 156.21 0)
@@
 		(on_board yes)
 		(dnp no)
-		(fields_autoplaced yes)
 		(property "Reference" "R407"
 			(at 76.2 154.9399 0)
@@
 		(on_board yes)
 		(dnp no)
-		(fields_autoplaced yes)
 		(property "Reference" "C2"
-			(at 275.59 117.2209 0)
+			(at 268.605 121.92 0)
 			(effects
 				(font
@@
 		)
 		(property "Value" "22µ 250V"
-			(at 275.59 119.7609 0)
+			(at 261.62 123.825 0)
 			(effects
 				(font
@@
 		(on_board yes)
 		(dnp no)
-		(fields_autoplaced yes)
 		(property "Reference" "C1"
-			(at 257.81 117.2209 0)
+			(at 254.635 114.935 0)
 			(effects
 				(font
@@
 		)
 		(property "Value" "22µ 250V"
-			(at 257.81 119.7609 0)
+			(at 254.635 116.84 0)
 			(effects
 				(font

Commit message: Major Final Update Finalize design check all changes made during review revert back Footprint of Inductor Split PCB design into two projects add some functionality to ESP32 (Bootstrap and crystal)
Parts:
- L401: footprint Inductor_THT:L_Toroid_Horizontal_D16.8mm_P14.70mm_Vishay_TJ3 -> Eigene:FT50-43
Changed lines of the file:
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@@
 			)
 		)
-		(property "Footprint" "Inductor_THT:L_Toroid_Horizontal_D16.8mm_P14.70mm_Vishay_TJ3"
+		(property "Footprint" "Eigene:FT50-43"
 			(at 73.66 129.54 0)
 			(effects
